Commit message: refine description and externalize robot parameters

File: urdf/marvin.urdf.xacro (robot description, xacro)
@@ -5,4 +5,7 @@
        xyz                  Translation offset from connected_to
        rpy                  Rotation offset from connected_to
+       mounts_file          YAML source for the bimanual mounting transforms
+       left_base_xyz/rpy    base_link -> Base_L mounting transform
+       right_base_xyz/rpy   base_link -> Base_R mounting transform
        ros2_control         Whether to include the <ros2_control> block
        use_fake_hardware    Use mock_components/GenericSystem (true) or real plugin
@@ -17,4 +20,10 @@
   <xacro:arg name="xyz" default="0 0 0"/>
   <xacro:arg name="rpy" default="0 0 0"/>
+  <xacro:arg name="mounts_file" default="$(find marvin_description)/config/arm_mounts.yaml"/>
+  <xacro:property name="arm_mounts" value="${xacro.load_yaml('$(arg mounts_file)')}"/>
+  <xacro:arg name="left_base_xyz" default="${arm_mounts['left_arm']['origin']['xyz']}"/>
+  <xacro:arg name="left_base_rpy" default="${arm_mounts['left_arm']['origin']['rpy']}"/>
+  <xacro:arg name="right_base_xyz" default="${arm_mounts['right_arm']['origin']['xyz']}"/>
+  <xacro:arg name="right_base_rpy" default="${arm_mounts['right_arm']['origin']['rpy']}"/>
   <xacro:arg name="ros2_control" default="true"/>
   <xacro:arg name="use_fake_hardware" default="true"/>
@@ -33,5 +42,9 @@
     connected_to="$(arg connected_to)"
     xyz="$(arg xyz)"
-    rpy="$(arg rpy)"/>
+    rpy="$(arg rpy)"
+    left_base_xyz="$(arg left_base_xyz)"
+    left_base_rpy="$(arg left_base_rpy)"
+    right_base_xyz="$(arg right_base_xyz)"
+    right_base_rpy="$(arg right_base_rpy)"/>
   <!-- ros2_control block (conditional) -->
   <xacro:if value="$(arg ros2_control)">

File: urdf/parts/marvin_arm.ros2_control.xacro (robot description, xacro)
@@ -1,6 +1,5 @@
 <?xml version="1.0"?>
 <!-- Marvin arm ros2_control block. Exposes 14 arm joints (7 per arm)
-     with reserved position/velocity/effort command interfaces and
-     position/velocity/effort state interfaces.
+     with position command interface and position/velocity/effort state interfaces.
      Defaults to mock_components/GenericSystem for fake-hardware validation. -->
 <robot xmlns:xacro="http://www.ros.org/wiki/xacro">
@@ -24,6 +23,4 @@
         <joint name="${joint_name}">
           <command_interface name="position"/>
-          <command_interface name="velocity"/>
-          <command_interface name="effort"/>
           <state_interface name="position"/>
           <state_interface name="velocity"/>

File: urdf/parts/marvin_bimanual_arm.xacro (robot description, xacro)
@@ -3,8 +3,16 @@
      and composes them into a single dual-arm assembly. -->
 <robot xmlns:xacro="http://ros.org/wiki/xacro">
+  <xacro:include filename="$(find marvin_description)/urdf/parts/marvin_arm_parameters.xacro"/>
   <xacro:include filename="$(find marvin_description)/urdf/parts/marvin_left_arm.xacro"/>
   <xacro:include filename="$(find marvin_description)/urdf/parts/marvin_right_arm.xacro"/>
   <xacro:macro name="marvin_bimanual_arm"
-    params="connected_to:='world' xyz:='0 0 0' rpy:='0 0 0' parent:=base_link">
+    params="connected_to:='world'
+            xyz:='0 0 0'
+            rpy:='0 0 0'
+            parent:=base_link
+            left_base_xyz:='0 0.037 0.140'
+            left_base_rpy:='-1.57 0 0'
+            right_base_xyz:='0 -0.037 0.140'
+            right_base_rpy:='1.57 0 0'">
     <xacro:unless value="${not connected_to}">
       <link name="${connected_to}"/>
@@ -15,6 +23,6 @@
       </joint>
     </xacro:unless>
-    <xacro:marvin_left_arm parent="${parent}"/>
-    <xacro:marvin_right_arm parent="${parent}"/>
+    <xacro:marvin_left_arm parent="${parent}" xyz="${left_base_xyz}" rpy="${left_base_rpy}"/>
+    <xacro:marvin_right_arm parent="${parent}" xyz="${right_base_xyz}" rpy="${right_base_rpy}"/>
   </xacro:macro>
 </robot>

File: urdf/parts/marvin_left_arm.xacro (robot description, xacro)
@@ -6,5 +6,5 @@
 <robot xmlns:xacro="http://ros.org/wiki/xacro">
   <xacro:macro name="marvin_left_arm"
-    params="parent:=base_link xyz:='0 0.037 0.140' rpy:='-1.57 0 0' description_pkg:=marvin_description">
+    params="parent:=base_link xyz:='0 0 0' rpy:='0 0 0' description_pkg:=marvin_description">
     <!-- Mounting joint from parent (typically base_link) to Base_L -->
     <joint name="base_to_left_arm" type="fixed">
@@ -15,18 +15,5 @@
     <link
       name="Base_L">
-      <inertial>
-        <origin
-          xyz="0.00032267 4.798E-05 0.04066353"
-          rpy="0 0 0" />
-        <mass
-          value="1.1962" />
-        <inertia
-          ixx="0.00107329"
-          ixy="-1.68E-06"
-          ixz="-1.05E-05"
-          iyy="0.00107003"
-          iyz="-3.43E-06"
-          izz="0.00127315" />
-      </inertial>
+      <xacro:marvin_link_inertial key="base"/>
       <visual>
         <origin
@@ -53,18 +40,5 @@
     <link
       name="Link1_L">
-      <inertial>
-        <origin
-          xyz="0.00002347 0.00557150 -0.03075998"
-          rpy="0 0 0" />
-        <mass
-          value="1.9705" />
-        <inertia
-          ixx="0.00492293"
-          ixy="0.00000550"
-          ixz="0.00000193"
-          iyy="0.00526513"
-          iyz="0.00033232"
-          izz="0.00188107" />
-      </inertial>
+      <xacro:marvin_link_inertial key="link1"/>
       <visual>
         <origin
@@ -92,35 +66,13 @@
       name="Joint1_L"
       type="revolute">
-      <origin
-        xyz="0 0 0.1745"
-        rpy="0 0 0" />
+      <xacro:marvin_joint_parameters key="joint1"/>
       <parent
         link="Base_L" />
       <child
         link="Link1_L" />
-      <axis
-        xyz="0 0 1" />
-      <limit
-        lower="-2.9671"
-        upper="2.9671"
-        effort="108"
-        velocity="3.1416" />
     </joint>
     <link
       name="Link2_L">
-      <inertial>
-        <origin
-          xyz="0.00013483 0.06170460 0.00950639"
-          rpy="0 0 0" />
-        <mass
-          value="2.24398" />
-        <inertia
-          ixx="0.01194933"
-          ixy="0.00000336"
-          ixz="0.00000091"
-          iyy="0.00361581"
-          iyz="-0.00132804"
-          izz="0.01098356" />
-      </inertial>
+      <xacro:marvin_link_inertial key="link2"/>
       <visual>
         <origin
@@ -148,35 +100,13 @@
       name="Joint2_L"
       type="revolute">
-      <origin
-        xyz="0 0 0"
-        rpy="1.5708 0 0" />
+      <xacro:marvin_joint_parameters key="joint2"/>
       <parent
         link="Link1_L" />
       <child
         link="Link2_L" />
-      <axis
-        xyz="0 0 1" />
-      <limit
-        lower="-2.0944"
-        upper="2.0944"
-        effort="108"
-        velocity="3.1416" />
     </joint>
     <link
       name="Link3_L">
-      <inertial>
-        <origin
-          xyz="0.00968562 0.00246599 -0.04627302"
-          rpy="0 0 0" />
-        <mass
-          value="1.9242" />
-        <inertia
-          ixx="0.00718224"
-          ixy="0.00004413"
-          ixz="0.00089552"
-          iyy="0.00762563"
-          iyz="0.00022096"
-          izz="0.00178597" />
-      </inertial>
+      <xacro:marvin_link_inertial key="link3"/>
       <visual>
         <origin
@@ -202,35 +132,13 @@
       name="Joint3_L"
       type="revolute">
-      <origin
-        xyz="0 0.287 0"
-        rpy="-1.5708 0 0" />
+      <xacro:marvin_joint_parameters key="joint3"/>
       <parent
         link="Link2_L" />
       <child
         link="Link3_L" />
-      <axis
-        xyz="0 0 1" />
-      <limit
-        lower="-2.9671"
-        upper="2.9671"
-        effort="66"
-        velocity="3.1416" />
     </joint>
     <link
       name="Link4_L">
-      <inertial>
-        <origin
-          xyz="0.00850411 -0.04718223 0.00941509"
-          rpy="0 0 0" />
-        <mass
-          value="1.6085" />
-        <inertia
-          ixx="0.00580480"
-          ixy="-0.00066669"
-          ixz="-0.00012722"
-          iyy="0.00223807"
-          iyz="0.00070523"
-          izz="0.00533060" />
-      </inertial>
+      <xacro:marvin_link_inertial key="link4"/>
       <visual>
         <origin
@@ -256,35 +164,13 @@
       name="Joint4_L"
       type="revolute">
-      <origin
-        xyz="0.018 0 0"
-        rpy="-1.5708 0 3.1416" />
+      <xacro:marvin_joint_parameters key="joint4"/>
       <parent
         link="Link3_L" />
       <child
         link="Link4_L" />
-      <axis
-        xyz="0 0 1" />
-      <limit
-        lower="-2.5307"
-        upper="1.0472"
-        effort="66"
-        velocity="3.1416" />
     </joint>
     <link
       name="Link5_L">
-      <inertial>
-        <origin
-          xyz="0.00051127 0.00101064 -0.11271739"
-          rpy="0 0 0" />
-        <mass
-          value="2.0883" />
-        <inertia
-          ixx="0.00626603"
-          ixy="0.00004009"
-          ixz="0.00005338"
-          iyy="0.00564387"
-          iyz="-0.00006193"
-          izz="0.00243632" />
-      </inertial>
+      <xacro:marvin_link_inertial key="link5_left"/>
       <visual>
         <origin
@@ -310,35 +196,13 @@
       name="Joint5_L"
       type="revolute">
-      <origin
-        xyz="0.018 -0.314 0"
-        rpy="-1.5708 0 3.1416" />
+      <xacro:marvin_joint_parameters key="joint5"/>
       <parent
         link="Link4_L" />
       <child
         link="Link5_L" />
-      <axis
-        xyz="0 0 1" />
-      <limit
-        lower="-2.9671"
-        upper="2.9671"
-        effort="18"
-        velocity="3.1416" />
     </joint>
     <link
       name="Link6_L">
-      <inertial>
-        <origin
-          xyz="0.00032659 0.00531336 -0.00030182"
-          rpy="0 0 0" />
-        <mass
-          value="0.72496" />
-        <inertia
-          ixx="0.00046040"
-          ixy="0.00000189"
-          ixz="0.00000083"
-          iyy="0.00051716"
-          iyz="-0.00000346"
-          izz="0.00042521" />
-      </inertial>
+      <xacro:marvin_link_inertial key="link6_left"/>
       <visual>
         <origin
@@ -364,35 +228,13 @@
       name="Joint6_L"
       type="revolute">
-      <origin
-        xyz="0 0 0"
-        rpy="1.5708 -1.5708 0" />
+      <xacro:marvin_joint_parameters key="joint6"/>
       <parent
         link="Link5_L" />
       <child
         link="Link6_L" />
-      <axis
-        xyz="0 0 1" />
-      <limit
-        lower="-1.0472"
-        upper="1.0472"
-        effort="18"
-        velocity="3.1416" />
     </joint>
     <link
       name="Link7_L">
-      <inertial>
-        <origin
-          xyz="-0.00009108 -0.03153255 0.00889371"
-          rpy="0 0 0" />
-        <mass
-          value="0.68606" />
-        <inertia
-          ixx="0.00173687"
-          ixy="-0.00000345"
-          ixz="-0.00000116"
-          iyy="0.00089035"
-          iyz="0.00030680"
-          izz="0.00139406" />
-      </inertial>
+      <xacro:marvin_link_inertial key="link7"/>
       <visual>
         <origin
@@ -418,22 +260,15 @@
       name="Joint7_L"
       type="revolute">
-      <origin
-        xyz="0 0 0"
-        rpy="1.5708 -1.5708 0" />
+      <xacro:marvin_joint_parameters key="joint7"/>
       <parent
         link="Link6_L" />
       <child
         link="Link7_L" />
-      <axis
-        xyz="0 0 1" />
-      <limit
-        lower="-1.5708"
-        upper="1.5708"
-        effort="18"
-        velocity="3.1416" />
     </joint>
     <link name="flange_L"/>
     <joint name="joint_flange_L" type="fixed">
-      <origin xyz="0.0 -0.095 0.0" rpy="1.5708 -1.5708 0" />
+      <origin
+        xyz="${marvin_kinematics['flange']['origin']['xyz']}"
+        rpy="${marvin_kinematics['flange']['origin']['rpy']}"/>
       <parent link="Link7_L" />
       <child link="flange_L" />

File: urdf/parts/marvin_right_arm.xacro (robot description, xacro)
@@ -6,5 +6,5 @@
 <robot xmlns:xacro="http://ros.org/wiki/xacro">
   <xacro:macro name="marvin_right_arm"
-    params="parent:=base_link xyz:='0 -0.037 0.140' rpy:='1.57 0 0' description_pkg:=marvin_description">
+    params="parent:=base_link xyz:='0 0 0' rpy:='0 0 0' description_pkg:=marvin_description">
     <!-- Mounting joint from parent (typically base_link) to Base_R -->
     <joint name="base_to_right_arm" type="fixed">
@@ -15,18 +15,5 @@
     <link
       name="Base_R">
-      <inertial>
-        <origin
-          xyz="0.00032267 4.798E-05 0.04066353"
-          rpy="0 0 0" />
-        <mass
-          value="1.1962" />
-        <inertia
-          ixx="0.00107329"
-          ixy="-1.68E-06"
-          ixz="-1.05E-05"
-          iyy="0.00107003"
-          iyz="-3.43E-06"
-          izz="0.00127315" />
-      </inertial>
+      <xacro:marvin_link_inertial key="base"/>
       <visual>
         <origin
@@ -53,18 +40,5 @@
     <link
       name="Link1_R">
-      <inertial>
-        <origin
-          xyz="0.00002347 0.00557150 -0.03075998"
-          rpy="0 0 0" />
-        <mass
-          value="1.9705" />
-        <inertia
-          ixx="0.00492293"
-          ixy="0.00000550"
-          ixz="0.00000193"
-          iyy="0.00526513"
-          iyz="0.00033232"
-          izz="0.00188107" />
-      </inertial>
+      <xacro:marvin_link_inertial key="link1"/>
       <visual>
         <origin
@@ -92,35 +66,13 @@
       name="Joint1_R"
       type="revolute">
-      <origin
-        xyz="0 0 0.1745"
-        rpy="0 0 0" />
+      <xacro:marvin_joint_parameters key="joint1"/>
       <parent
         link="Base_R" />
       <child
         link="Link1_R" />
-      <axis
-        xyz="0 0 1" />
-      <limit
-        lower="-2.9671"
-        upper="2.9671"
-        effort="108"
-        velocity="3.1416" />
     </joint>
     <link
       name="Link2_R">
-      <inertial>
-        <origin
-          xyz="0.00013483 0.06170460 0.00950639"
-          rpy="0 0 0" />
-        <mass
-          value="2.24398" />
-        <inertia
-          ixx="0.01194933"
-          ixy="0.00000336"
-          ixz="0.00000091"
-          iyy="0.00361581"
-          iyz="-0.00132804"
-          izz="0.01098356" />
-      </inertial>
+      <xacro:marvin_link_inertial key="link2"/>
       <visual>
         <origin
@@ -148,35 +100,13 @@
       name="Joint2_R"
       type="revolute">
-      <origin
-        xyz="0 0 0"
-        rpy="1.5708 0 0" />
+      <xacro:marvin_joint_parameters key="joint2"/>
       <parent
         link="Link1_R" />
       <child
         link="Link2_R" />
-      <axis
-        xyz="0 0 1" />
-      <limit
-        lower="-2.0944"
-        upper="2.0944"
-        effort="108"
-        velocity="3.1416" />
     </joint>
     <link
       name="Link3_R">
-      <inertial>
-        <origin
-          xyz="0.00968562 0.00246599 -0.04627302"
-          rpy="0 0 0" />
-        <mass
-          value="1.9242" />
-        <inertia
-          ixx="0.00718224"
-          ixy="0.00004413"
-          ixz="0.00089552"
-          iyy="0.00762563"
-          iyz="0.00022096"
-          izz="0.00178597" />
-      </inertial>
+      <xacro:marvin_link_inertial key="link3"/>
       <visual>
         <origin
@@ -202,35 +132,13 @@
       name="Joint3_R"
       type="revolute">
-      <origin
-        xyz="0 0.287 0"
-        rpy="-1.5708 0 0" />
+      <xacro:marvin_joint_parameters key="joint3"/>
       <parent
         link="Link2_R" />
       <child
         link="Link3_R" />
-      <axis
-        xyz="0 0 1" />
-      <limit
-        lower="-2.9671"
-        upper="2.9671"
-        effort="66"
-        velocity="3.1416" />
     </joint>
     <link
       name="Link4_R">
-      <inertial>
-        <origin
-          xyz="0.00850411 -0.04718223 0.00941509"
-          rpy="0 0 0" />
-        <mass
-          value="1.6085" />
-        <inertia
-          ixx="0.00580480"
-          ixy="-0.00066669"
-          ixz="-0.00012722"
-          iyy="0.00223807"
-          iyz="0.00070523"
-          izz="0.00533060" />
-      </inertial>
+      <xacro:marvin_link_inertial key="link4"/>
       <visual>
         <origin
@@ -256,35 +164,13 @@
       name="Joint4_R"
       type="revolute">
-      <origin
-        xyz="0.018 0 0"
-        rpy="-1.5708 0 3.1416" />
+      <xacro:marvin_joint_parameters key="joint4"/>
       <parent
         link="Link3_R" />
       <child
         link="Link4_R" />
-      <axis
-        xyz="0 0 1" />
-      <limit
-        lower="-2.5307"
-        upper="1.0472"
-        effort="66"
-        velocity="3.1416" />
     </joint>
     <link
       name="Link5_R">
-      <inertial>
-        <origin
-          xyz="-0.00051127 -0.00101064 -0.11271739"
-          rpy="0 0 0" />
-        <mass
-          value="2.0883" />
-        <inertia
-          ixx="0.00626603"
-          ixy="0.00004009"
-          ixz="-0.00005338"
-          iyy="0.00564387"
-          iyz="0.00006193"
-          izz="0.00243632" />
-      </inertial>
+      <xacro:marvin_link_inertial key="link5_right"/>
       <visual>
         <origin
@@ -310,35 +196,13 @@
       name="Joint5_R"
       type="revolute">
-      <origin
-        xyz="0.018 -0.314 0"
-        rpy="-1.5708 0 3.1416" />
+      <xacro:marvin_joint_parameters key="joint5"/>
       <parent
         link="Link4_R" />
       <child
         link="Link5_R" />
-      <axis
-        xyz="0 0 1" />
-      <limit
-        lower="-2.9671"
-        upper="2.9671"
-        effort="18"
-        velocity="3.1416" />
     </joint>
     <link
       name="Link6_R">
-      <inertial>
-        <origin
-          xyz="0.00032659 -0.00531336 0.00030182"
-          rpy="0 0 0" />
-        <mass
-          value="0.72496" />
-        <inertia
-          ixx="0.00046040"
-          ixy="-0.00000189"
-          ixz="-0.00000083"
-          iyy="0.00051716"
-          iyz="-0.00000346"
-          izz="0.00042521" />
-      </inertial>
+      <xacro:marvin_link_inertial key="link6_right"/>
       <visual>
         <origin
@@ -364,35 +228,13 @@
       name="Joint6_R"
       type="revolute">
-      <origin
-        xyz="0 0 0"
-        rpy="1.5708 -1.5708 0" />
+      <xacro:marvin_joint_parameters key="joint6"/>
       <parent
         link="Link5_R" />
       <child
         link="Link6_R" />
-      <axis
-        xyz="0 0 1" />
-      <limit
-        lower="-1.0472"
-        upper="1.0472"
-        effort="18"
-        velocity="3.1416" />
     </joint>
     <link
       name="Link7_R">
-      <inertial>
-        <origin
-          xyz="-0.00009108 -0.03153255 0.00889371"
-          rpy="0 0 0" />
-        <mass
-          value="0.68606" />
-        <inertia
-          ixx="0.00173687"
-          ixy="-0.00000345"
-          ixz="-0.00000116"
-          iyy="0.00089035"
-          iyz="0.00030680"
-          izz="0.00139406" />
-      </inertial>
+      <xacro:marvin_link_inertial key="link7"/>
       <visual>
         <origin
@@ -418,22 +260,15 @@
       name="Joint7_R"
       type="revolute">
-      <origin
-        xyz="0 0 0"
-        rpy="1.5708 -1.5708 0" />
+      <xacro:marvin_joint_parameters key="joint7"/>
       <parent
         link="Link6_R" />
       <child
         link="Link7_R" />
-      <axis
-        xyz="0 0 1" />
-      <limit
-        lower="-1.5708"
-        upper="1.5708"
-        effort="18"
-        velocity="3.1416" />
     </joint>
     <link name="flange_R"/>
     <joint name="joint_flange_R" type="fixed">
-      <origin xyz="0.0 -0.095 0.0" rpy="1.5708 -1.5708 0" />
+      <origin
+        xyz="${marvin_kinematics['flange']['origin']['xyz']}"
+        rpy="${marvin_kinematics['flange']['origin']['rpy']}"/>
       <parent link="Link7_R" />
       <child link="flange_R" />
