Commit message: adjust stand link radius

File: urdf/parts/marvin_stand.xacro (robot description, xacro)
@@ -52,5 +52,5 @@
         rpy="0 0 0" />
       <geometry>
-        <cylinder radius="0.090" length="1.0"/>
+        <cylinder radius="0.060" length="1.0"/>
       </geometry>
     </visual>
@@ -60,5 +60,5 @@
         rpy="0 0 0" />
       <geometry>
-        <cylinder radius="0.090" length="1.0"/>
+        <cylinder radius="0.060" length="1.0"/>
       </geometry>
     </collision>
